File: Choc40.kicad_sch (KiCad schematic)
At the start: 0 parts

Commit message: Added Type C.pretty
https://github.com/ai03-2725/Type-C.pretty.git
Parts:
- added C1: 1uF, Capacitor_SMD:C_0603_1608Metric, symbol Device:C_Small
- added C2, C3: 0.1uF, Capacitor_SMD:C_0603_1608Metric, symbol Device:C_Small
- added C4: 10uF, Capacitor_SMD:C_0603_1608Metric, symbol Device:C_Small
- added C5: 4.7n, Capacitor_SMD:C_0603_1608Metric, symbol Device:C_Small
- added D1, D10, D11, D12, D13, D14, D15, D16, D17, D18, D19, D2, D20, D21, D22, D23, D24, D25, D26, D27, D28, D29, D3, D30, D31, D32, D33, D34, D35, D36, D37, D38, D39, D4, D40, D5, D6, D7, D8, D9: D_Small, Diode_SMD:D_SOD-123, symbol Device:D_Small
- added D41: PRTR5V0U2X, Package_TO_SOT_SMD:SOT-143, symbol Power_Protection:PRTR5V0U2X
- added F1: 500mA, Fuse:Fuse_1206_3216Metric, symbol Device:Polyfuse_Small
- added R1, R4: 10k, Resistor_SMD:R_0603_1608Metric, symbol Device:R_Small
- added R2, R3: 22, Resistor_SMD:R_0603_1608Metric, symbol Device:R_Small
- added R5, R6: 5k1, Resistor_SMD:R_0603_1608Metric, symbol Device:R_Small
- added R7: 1M, Resistor_SMD:R_0603_1608Metric, symbol Device:R_Small
- added SW1, SW10, SW11, SW12, SW14, SW15, SW16, SW17, SW18, SW19, SW2, SW20, SW21, SW22, SW25, SW26, SW27, SW28, SW29, SW3, SW30, SW31, SW32, SW33a1, SW34b1, SW36, SW37, SW4, SW5, SW6, SW7, SW8, SW9: SW_Push, mbk:Choc-1u-solder, symbol Switch:SW_Push
- added SW13, SW33b1, SW34a1, SW35, SW39, SW40: SW_Push, mbk:Choc-1.25u-solder, symbol Switch:SW_Push
- added SW23, SW24: SW_Push, mbk:Choc-1.75u-solder, symbol Switch:SW_Push
- added SW38: SW_Push, mbk:Choc-6.25u-solder, symbol Switch:SW_Push
- added SW99: SW_Push, random-keyboard-parts:SKQG-1155865, symbol Switch:SW_Push
- added U1: ATmega32U2-MU, Package_DFN_QFN:QFN-32-1EP_5x5mm_P0.5mm_EP3.1x3.1mm, symbol MCU_Microchip_ATmega:ATmega32U2-MU
- added USB1: HRO-TYPE-C-31-M-12, Type-C:HRO-TYPE-C-31-M-12, symbol Type-C:HRO-TYPE-C-31-M-12
- added Y1: Resonator_Small, Crystal:Resonator_SMD_muRata_CSTxExxV-3Pin_3.0x1.1mm, symbol Device:Resonator_Small
Connections:
- new net: R4.2, U1.13 (~HWB~/PD7)
- new net: R1.2, SW99.2, U1.24 (PC1/~RESET)
- new net: U1.1 (XTAL1), Y1.1
- new net: U1.2 (PC0/XTAL2), Y1.3
- new net: R6.1, USB1.10 (CC2)
- new net: C5.2, R7.1, USB1.13 (SHIELD)
- new net: R5.1, USB1.4 (CC1)
- new net: C1.1, U1.27 (UCAP)
- new net: D30.2 (A), SW30.1
- new net: D18.2 (A), SW18.1
- new net: SW18.2, SW29.2, SW38.2, SW6.2
- new net: D37.2 (A), SW37.1
- new net: D33.2 (A), SW33a1.1, SW33b1.1
- new net: SW10.2, SW22.2, SW33a1.2, SW33b1.2
- new net: D26.2 (A), SW26.1
- new net: SW15.2, SW26.2, SW3.2, SW36.2
- new net: D34.2 (A), SW34a1.1, SW34b1.1
- new net: SW12.2, SW34a1.2, SW34b1.2, SW40.2
- new net: D3.2 (A), SW3.1
- new net: D39.2 (A), SW39.1
- new net: SW11.2, SW23.2, SW39.2
- new net: D4.2 (A), SW4.1
- new net: SW16.2, SW27.2, SW37.2, SW4.2
- new net: D32.2 (A), SW32.1
- new net: SW21.2, SW32.2, SW9.2
- new net: D24.2 (A), SW24.1
- new net: D14.2 (A), SW14.1
- new net: SW14.2, SW2.2, SW25.2
- new net: D22.2 (A), SW22.1
- new net: D6.2 (A), SW6.1
- new net: D11.2 (A), SW11.1
- new net: D25.2 (A), SW25.1
- new net: D38.2 (A), SW38.1
- new net: D40.2 (A), SW40.1
- new net: D28.2 (A), SW28.1
- new net: SW17.2, SW28.2, SW5.2
- new net: D36.2 (A), SW36.1
- new net: D27.2 (A), SW27.1
- new net: D8.2 (A), SW8.1
- new net: D31.2 (A), SW31.1
- new net: D21.2 (A), SW21.1
- new net: D15.2 (A), SW15.1
- new net: SW19.2, SW30.2, SW7.2
- new net: D12.2 (A), SW12.1
- new net: D20.2 (A), SW20.1
- new net: SW20.2, SW31.2, SW8.2
- new net: D16.2 (A), SW16.1
- new net: D19.2 (A), SW19.1
- new net: D29.2 (A), SW29.1
- new net: D7.2 (A), SW7.1
- new net: D23.2 (A), SW23.1
- new net: SW1.2, SW13.2, SW24.2, SW35.2
- new net: D9.2 (A), SW9.1
- new net: D10.2 (A), SW10.1
- new net: D13.2 (A), SW13.1
- new net: D17.2 (A), SW17.1
- new net: D35.2 (A), SW35.1
- new net: D5.2 (A), SW5.1
- new net: D2.2 (A), SW2.1
- new net: D1.2 (A), SW1.1
- new net +5V: C2.1, C3.1, C4.1, F1.1, R1.1, U1.31 (UVCC), U1.32 (AVCC), U1.4 (VCC)
- new net D+: D41.3 (I/O2), R2.2, USB1.6 (DP1), USB1.8 (DP2)
- new net D-: D41.2 (I/O1), R3.2, USB1.5 (DN2), USB1.7 (DN1)
- new net DP+: R2.1, U1.29 (D+)
- new net DP-: R3.1, U1.30 (D-)
- new net GND: C1.2, C2.2, C3.2, C4.2, C5.1, D41.1 (GND), R4.1, R5.2, R6.2, R7.2, SW99.1, U1.28 (UGND), U1.3 (GND), U1.33 (GND), USB1.1 (GND), USB1.12 (GND), Y1.2
- new net VCC: D41.4 (VCC), F1.2, USB1.11 (VBUS), USB1.2 (VBUS)
- new net row0: D1.1 (K), D10.1 (K), D11.1 (K), D12.1 (K), D2.1 (K), D3.1 (K), D4.1 (K), D5.1 (K), D6.1 (K), D7.1 (K), D8.1 (K), D9.1 (K)
- new net row1: D13.1 (K), D14.1 (K), D15.1 (K), D16.1 (K), D17.1 (K), D18.1 (K), D19.1 (K), D20.1 (K), D21.1 (K), D22.1 (K), D23.1 (K)
- new net row2: D24.1 (K), D25.1 (K), D26.1 (K), D27.1 (K), D28.1 (K), D29.1 (K), D30.1 (K), D31.1 (K), D32.1 (K), D33.1 (K), D34.1 (K)
- new net row3: D35.1 (K), D36.1 (K), D37.1 (K), D38.1 (K), D39.1 (K), D40.1 (K)
- no-connect marks 0 -> 2
