File: Choc40.kicad_sch (KiCad schematic)
At the start: 100 parts, among them SW1 SW_Push, SW10 SW_Push, SW11 SW_Push, SW12 SW_Push, SW13 SW_Push, SW14 SW_Push, SW15 SW_Push, SW16 SW_Push, SW17 SW_Push, SW18 SW_Push, SW19 SW_Push, SW2 SW_Push, SW20 SW_Push, SW21 SW_Push, SW22 SW_Push, SW23 SW_Push, SW24 SW_Push, SW25 SW_Push, SW26 SW_Push, SW27 SW_Push, SW28 SW_Push, SW29 SW_Push, SW3 SW_Push, SW30 SW_Push, SW31 SW_Push, SW32 SW_Push, SW33a1 SW_Push, SW33b1 SW_Push, SW34a1 SW_Push, SW34b1 SW_Push, SW35 SW_Push, SW36 SW_Push, SW37 SW_Push, SW38 SW_Push, SW39 SW_Push, SW4 SW_Push, SW40 SW_Push, SW5 SW_Push, SW6 SW_Push, SW7 SW_Push, SW8 SW_Push, SW9 SW_Push, SW99 SW_Push, U1 ATmega32U2-MU, Y1 Resonator_Small

Commit message: le epic progression
Connections:
- net row0: no longer D12.1 (K)
- net row3: now also D12.1 (K), U1.12 (PD6)
- net col5: now reaches SW18.2, SW29.2, SW38.2, SW6.2
- net col9: now reaches SW10.2, SW22.2, SW33a1.2, SW33b1.2
- net col9: now also SW40.2
- net col2: now reaches SW15.2, SW26.2, SW3.2
- net col2: now also SW37.2; no longer SW36.2
- net col10: now reaches SW12.2, SW34a1.2, SW34b1.2
- net col10: now also SW11.2, SW23.2; no longer SW40.2
- net col3: now reaches SW16.2, SW27.2, SW4.2
- net col3: no longer SW37.2
- net col8: now reaches SW21.2, SW32.2, SW9.2
- net col8: now also SW39.2
- net col1: now reaches SW14.2, SW2.2, SW25.2
- net col1: now also SW36.2
- net col4: now reaches SW17.2, SW28.2, SW5.2
- net col6: now reaches SW19.2, SW30.2, SW7.2
- net col7: now reaches SW20.2, SW31.2, SW8.2
- net col0: now reaches SW1.2, SW13.2, SW24.2, SW35.2
Other:
- moved on the sheet: D12, D34, D36, D37, D39, D40, SW12, SW34a1, SW34b1, SW36, SW37, SW39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
