File: Choc40.kicad_pcb (KiCad board)
At the start: 0 parts

Commit message: pcb go brr
Parts:
- added C1: 1uF, Capacitor_SMD:C_0603_1608Metric, B.Cu at (150.2, 107.0)
- added C2: 0.1uF, Capacitor_SMD:C_0603_1608Metric, B.Cu at (150.2, 110.0)
- added C3: 0.1uF, Capacitor_SMD:C_0603_1608Metric, B.Cu at (140.8, 107.5)
- added C4: 10uF, Capacitor_SMD:C_0603_1608Metric, B.Cu at (129.3, 103.5)
- added C5: 4.7n, Capacitor_SMD:C_0603_1608Metric, B.Cu at (145.6, 104.4)
- added D1: D_Small, Diode_SMD:D_SOD-123, B.Cu at (38.7, 39.4)
- added D10: D_Small, Diode_SMD:D_SOD-123, B.Cu at (200.7, 39.4)
- added D11: D_Small, Diode_SMD:D_SOD-123, B.Cu at (218.7, 39.4)
- added D12: D_Small, Diode_SMD:D_SOD-123, B.Cu at (236.7, 39.4)
- added D13: D_Small, Diode_SMD:D_SOD-123, B.Cu at (41.0, 56.4)
- added D14: D_Small, Diode_SMD:D_SOD-123, B.Cu at (61.2, 56.4)
- added D15: D_Small, Diode_SMD:D_SOD-123, B.Cu at (79.2, 56.4)
- added D16: D_Small, Diode_SMD:D_SOD-123, B.Cu at (97.2, 56.4)
- added D17: D_Small, Diode_SMD:D_SOD-123, B.Cu at (115.2, 56.4)
- added D18: D_Small, Diode_SMD:D_SOD-123, B.Cu at (133.2, 56.4)
- added D19: D_Small, Diode_SMD:D_SOD-123, B.Cu at (151.2, 56.4)
- added D2: D_Small, Diode_SMD:D_SOD-123, B.Cu at (56.7, 39.4)
- added D20: D_Small, Diode_SMD:D_SOD-123, B.Cu at (169.2, 56.4)
- added D21: D_Small, Diode_SMD:D_SOD-123, B.Cu at (187.2, 56.4)
- added D22: D_Small, Diode_SMD:D_SOD-123, B.Cu at (205.2, 56.4)
- added D23: D_Small, Diode_SMD:D_SOD-123, B.Cu at (230.0, 56.4)
- added D24: D_Small, Diode_SMD:D_SOD-123, B.Cu at (45.4, 73.4)
- added D25: D_Small, Diode_SMD:D_SOD-123, B.Cu at (70.2, 73.4)
- added D26: D_Small, Diode_SMD:D_SOD-123, B.Cu at (88.2, 73.4)
- added D27: D_Small, Diode_SMD:D_SOD-123, B.Cu at (106.2, 73.4)
- added D28: D_Small, Diode_SMD:D_SOD-123, B.Cu at (124.2, 73.4)
- added D29: D_Small, Diode_SMD:D_SOD-123, B.Cu at (142.2, 73.4)
- added D3: D_Small, Diode_SMD:D_SOD-123, B.Cu at (74.7, 39.4)
- added D30: D_Small, Diode_SMD:D_SOD-123, B.Cu at (160.2, 73.4)
- added D31: D_Small, Diode_SMD:D_SOD-123, B.Cu at (178.2, 73.4)
- added D32: D_Small, Diode_SMD:D_SOD-123, B.Cu at (196.2, 73.4)
- added D33: D_Small, Diode_SMD:D_SOD-123, B.Cu at (216.5, 73.4)
- added D34: D_Small, Diode_SMD:D_SOD-123, B.Cu at (234.5, 73.4)
- added D35: D_Small, Diode_SMD:D_SOD-123, B.Cu at (41.0, 90.4)
- added D36: D_Small, Diode_SMD:D_SOD-123, B.Cu at (61.2, 90.4)
- added D37: D_Small, Diode_SMD:D_SOD-123, B.Cu at (79.2, 90.4)
- added D38: D_Small, Diode_SMD:D_SOD-123, B.Cu at (144.4, 90.4)
- added D39: D_Small, Diode_SMD:D_SOD-123, B.Cu at (212.0, 90.4)
- added D4: D_Small, Diode_SMD:D_SOD-123, B.Cu at (92.7, 39.4)
- added D40: D_Small, Diode_SMD:D_SOD-123, B.Cu at (234.6, 90.4)
- added D41: PRTR5V0U2X, Package_TO_SOT_SMD:SOT-143, B.Cu at (133.0, 33.5)
- added D5: D_Small, Diode_SMD:D_SOD-123, B.Cu at (110.7, 39.4)
- added D6: D_Small, Diode_SMD:D_SOD-123, B.Cu at (128.7, 39.4)
- added D7: D_Small, Diode_SMD:D_SOD-123, B.Cu at (146.7, 39.4)
- added D8: D_Small, Diode_SMD:D_SOD-123, B.Cu at (164.7, 39.4)
- added D9: D_Small, Diode_SMD:D_SOD-123, B.Cu at (182.7, 39.4)
- added F1: 500mA, Fuse:Fuse_1206_3216Metric, B.Cu at (139.0, 33.5)
- added R1: 10k, Resistor_SMD:R_0603_1608Metric, B.Cu at (150.2, 98.2)
- added R2: 22, Resistor_SMD:R_0603_1608Metric, B.Cu at (150.2, 101.2)
- added R3: 22, Resistor_SMD:R_0603_1608Metric, B.Cu at (150.2, 104.1)
- added R4: 10k, Resistor_SMD:R_0603_1608Metric, B.Cu at (124.9, 103.2)
- added R5: 5k1, Resistor_SMD:R_0603_1608Metric, B.Cu at (124.4, 100.2)
- added R6: 5k1, Resistor_SMD:R_0603_1608Metric, B.Cu at (129.3, 106.5)
- added R7: 1M, Resistor_SMD:R_0603_1608Metric, B.Cu at (128.9, 100.2)
- added SW1: SW_Push, mbk:Choc-1u-solder, F.Cu at (34.0, 33.5)
- added SW10: SW_Push, mbk:Choc-1u-solder, F.Cu at (196.0, 33.5)
- added SW11: SW_Push, mbk:Choc-1u-solder, F.Cu at (214.0, 33.5)
- added SW12: SW_Push, mbk:Choc-1u-solder, F.Cu at (232.0, 33.5)
- added SW13: SW_Push, mbk:Choc-1.25u-solder, F.Cu at (36.2, 50.5)
- added SW14: SW_Push, mbk:Choc-1u-solder, F.Cu at (56.5, 50.5)
- added SW15: SW_Push, mbk:Choc-1u-solder, F.Cu at (74.5, 50.5)
- added SW16: SW_Push, mbk:Choc-1u-solder, F.Cu at (92.5, 50.5)
- added SW17: SW_Push, mbk:Choc-1u-solder, F.Cu at (110.5, 50.5)
- added SW18: SW_Push, mbk:Choc-1u-solder, F.Cu at (128.5, 50.5)
- added SW19: SW_Push, mbk:Choc-1u-solder, F.Cu at (146.5, 50.5)
- added SW2: SW_Push, mbk:Choc-1u-solder, F.Cu at (52.0, 33.5)
- added SW20: SW_Push, mbk:Choc-1u-solder, F.Cu at (164.5, 50.5)
- added SW21: SW_Push, mbk:Choc-1u-solder, F.Cu at (182.5, 50.5)
- added SW22: SW_Push, mbk:Choc-1u-solder, F.Cu at (200.5, 50.5)
- added SW23: SW_Push, mbk:Choc-1.75u-solder, F.Cu at (225.2, 50.5)
- added SW24: SW_Push, mbk:Choc-1.75u-solder, F.Cu at (40.8, 67.5)
- added SW25: SW_Push, mbk:Choc-1u-solder, F.Cu at (65.5, 67.5)
- added SW26: SW_Push, mbk:Choc-1u-solder, F.Cu at (83.5, 67.5)
- added SW27: SW_Push, mbk:Choc-1u-solder, F.Cu at (101.5, 67.5)
- added SW28: SW_Push, mbk:Choc-1u-solder, F.Cu at (119.5, 67.5)
- added SW29: SW_Push, mbk:Choc-1u-solder, F.Cu at (137.5, 67.5)
- added SW3: SW_Push, mbk:Choc-1u-solder, F.Cu at (70.0, 33.5)
- added SW30: SW_Push, mbk:Choc-1u-solder, F.Cu at (155.5, 67.5)
- added SW31: SW_Push, mbk:Choc-1u-solder, F.Cu at (173.5, 67.5)
- added SW32: SW_Push, mbk:Choc-1u-solder, F.Cu at (191.5, 67.5)
- added SW33a1: SW_Push, mbk:Choc-1u-solder, F.Cu at (209.5, 67.5)
- added SW33b1: SW_Push, mbk:Choc-1.25u-solder, F.Cu at (211.8, 67.5)
- added SW34a1: SW_Push, mbk:Choc-1.25u-solder, F.Cu at (229.8, 67.5)
- added SW34b1: SW_Push, mbk:Choc-1u-solder, F.Cu at (227.5, 67.5)
- added SW35: SW_Push, mbk:Choc-1.25u-solder, F.Cu at (36.2, 84.5)
- added SW36: SW_Push, mbk:Choc-1u-solder, F.Cu at (56.5, 84.5)
- added SW37: SW_Push, mbk:Choc-1u-solder, F.Cu at (74.5, 84.5)
- added SW38: SW_Push, mbk:Choc-6.25u-solder, F.Cu at (139.8, 84.5)
- added SW39: SW_Push, mbk:Choc-1.25u-solder, F.Cu at (207.2, 84.5)
- added SW4: SW_Push, mbk:Choc-1u-solder, F.Cu at (88.0, 33.5)
- added SW40: SW_Push, mbk:Choc-1.25u-solder, F.Cu at (229.8, 84.5)
- added SW5: SW_Push, mbk:Choc-1u-solder, F.Cu at (106.0, 33.5)
- added SW6: SW_Push, mbk:Choc-1u-solder, F.Cu at (124.0, 33.5)
- added SW7: SW_Push, mbk:Choc-1u-solder, F.Cu at (142.0, 33.5)
- added SW8: SW_Push, mbk:Choc-1u-solder, F.Cu at (160.0, 33.5)
- added SW9: SW_Push, mbk:Choc-1u-solder, F.Cu at (178.0, 33.5)
- added SW99: SW_Push, random-keyboard-parts:SKQG-1155865, B.Cu at (160.0, 84.5)
- added U1: ATmega32U2-MU, Package_DFN_QFN:QFN-32-1EP_5x5mm_P0.5mm_EP3.1x3.1mm, B.Cu at (119.5, 84.5)
- added USB1: HRO-TYPE-C-31-M-12, Type-C:HRO-TYPE-C-31-M-12, B.Cu at (133.0, 20.9)
- added Y1: Resonator_Small, Crystal:Resonator_SMD_muRata_CSTxExxV-3Pin_3.0x1.1mm, B.Cu at (125.5, 83.0)
Routing:
- added copper zone on B.Cu, net GND
- added copper zone on F.Cu, net GND
Other:
- board outline added: 216 x 70.8 mm
- copper layers 0 -> 2
