File: Choc40.kicad_pcb (KiCad board)
At the start: 2 copper layers, 216 x 70.8 mm, 100 parts, among them SW1 SW_Push, SW10 SW_Push, SW11 SW_Push, SW12 SW_Push, SW13 SW_Push, SW14 SW_Push, SW15 SW_Push, SW16 SW_Push, SW17 SW_Push, SW18 SW_Push, SW19 SW_Push, SW2 SW_Push, SW20 SW_Push, SW21 SW_Push, SW22 SW_Push, SW23 SW_Push, SW24 SW_Push, SW25 SW_Push, SW26 SW_Push, SW27 SW_Push, SW28 SW_Push, SW29 SW_Push, SW3 SW_Push, SW30 SW_Push, SW31 SW_Push, SW32 SW_Push, SW33a1 SW_Push, SW33b1 SW_Push, SW34a1 SW_Push, SW34b1 SW_Push, SW35 SW_Push, SW36 SW_Push, SW37 SW_Push, SW38 SW_Push, SW39 SW_Push, SW4 SW_Push, SW40 SW_Push, SW5 SW_Push, SW6 SW_Push, SW7 SW_Push, SW8 SW_Push, SW9 SW_Push, SW99 SW_Push, U1 ATmega32U2-MU, Y1 Resonator_Small

Commit message: a
Parts:
- moved R6 81.0 mm to (142.0, 26.5), turned to 0 degrees
- moved C5 79.1 mm to (124.0, 28.2), turned to 0 degrees
- moved R5 73.7 mm to (124.0, 26.5)
- moved R7 73.2 mm to (142.0, 28.2), turned to 0 degrees
- moved R3 67.2 mm to (132.2, 39.4), turned to 90 degrees
- moved R2 63.9 mm to (133.8, 39.4), turned to 90 degrees
- moved C1 42.5 mm to (118.8, 78.5), turned to 90 degrees
- moved C2 34.3 mm to (125.5, 86.2), turned to 0 degrees
- moved C3 32.8 mm to (124.2, 79.2), turned to 0 degrees
- moved C4 26.3 mm to (121.2, 78.5), turned to 90 degrees
- moved R4 14.0 mm to (119.2, 90.4), turned to 90 degrees
- moved R1 11.7 mm to (154.2, 87.2), turned to 90 degrees
Routing:
- net Net-(D23-Pad2): track 0.00 -> 3.10 mm
- net Net-(D9-Pad2): track 0.00 -> 3.05 mm
- net Net-(D8-Pad2): track 0.00 -> 3.05 mm
- net Net-(D7-Pad2): track 0.00 -> 3.05 mm
- net Net-(D22-Pad2): track 0.00 -> 3.05 mm
- net Net-(D21-Pad2): track 0.00 -> 3.05 mm
- net Net-(D20-Pad2): track 0.00 -> 3.05 mm
- net Net-(D19-Pad2): track 0.00 -> 3.05 mm
- net Net-(D18-Pad2): track 0.00 -> 3.05 mm
- net Net-(D12-Pad2): track 0.00 -> 3.05 mm
- net Net-(D11-Pad2): track 0.00 -> 3.05 mm
- net Net-(D10-Pad2): track 0.00 -> 3.05 mm
- net Net-(D6-Pad2): track 0.00 -> 3.05 mm
- net Net-(D5-Pad2): track 0.00 -> 3.05 mm
- net Net-(D4-Pad2): track 0.00 -> 3.05 mm
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
Commit message: le epic progression
Parts:
- moved R1 1.55 mm to (154.2, 85.6), turned to -90 degrees
Connections:
- net Net-(SW1-Pad2) renamed col0
- net Net-(SW17-Pad2) renamed col4
- net Net-(SW18-Pad2) renamed col5
- net Net-(SW19-Pad2) renamed col6
- net Net-(SW20-Pad2) renamed col7
- D12 pad 1: row0 -> row3
- SW10 pad 2: Net-(SW10-Pad2) -> col9
- SW11 pad 2: Net-(SW11-Pad2) -> col10
- SW12 pad 2: Net-(SW12-Pad2) -> col10
- SW14 pad 2: Net-(SW14-Pad2) -> col1
- SW15 pad 2: Net-(SW15-Pad2) -> col2
- SW16 pad 2: Net-(SW16-Pad2) -> col3
- SW2 pad 2: Net-(SW14-Pad2) -> col1
- SW21 pad 2: Net-(SW21-Pad2) -> col8
- SW22 pad 2: Net-(SW10-Pad2) -> col9
- SW23 pad 2: Net-(SW11-Pad2) -> col10
- SW25 pad 2: Net-(SW14-Pad2) -> col1
- SW26 pad 2: Net-(SW15-Pad2) -> col2
- SW27 pad 2: Net-(SW16-Pad2) -> col3
- SW3 pad 2: Net-(SW15-Pad2) -> col2
- SW32 pad 2: Net-(SW21-Pad2) -> col8
- SW33a1 pad 2: Net-(SW10-Pad2) -> col9
- SW33b1 pad 2: Net-(SW10-Pad2) -> col9
- SW34a1 pad 2: Net-(SW12-Pad2) -> col10
- SW34b1 pad 2: Net-(SW12-Pad2) -> col10
- SW36 pad 2: Net-(SW15-Pad2) -> col1
- SW37 pad 2: Net-(SW16-Pad2) -> col2
- SW39 pad 2: Net-(SW11-Pad2) -> col8
- SW4 pad 2: Net-(SW16-Pad2) -> col3
- SW40 pad 2: Net-(SW12-Pad2) -> col9
- SW9 pad 2: Net-(SW21-Pad2) -> col8
- U1 pad 12: unconnected-(U1-Pad12) -> row3
Routing:
- net row3: track 0.00 -> 256.7 mm
- net row1: track 0.00 -> 200.8 mm, vias 0 -> 2
- net row2: track 0.00 -> 200.7 mm, vias 0 -> 2
- net row0: track 0.00 -> 196.1 mm, vias 0 -> 2
- net +5V: track 0.00 -> 102.8 mm, vias 0 -> 2
- net col9: track 0.00 -> 69.1 mm
- net col8: track 0.00 -> 66.8 mm
- net col1: track 0.00 -> 60.4 mm
- net col2: track 0.00 -> 60.3 mm
- net col10: track 0.00 -> 59.8 mm
- net col5: track 0.00 -> 57.5 mm
- net col0: track 0.00 -> 55.7 mm
- net DP+: track 0.00 -> 55.4 mm
- net DP-: track 0.00 -> 55.4 mm, vias 0 -> 2
- net Net-(R1-Pad2): track 0.00 -> 51.7 mm, vias 0 -> 2
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
Commit message: PCB finished
Parts:
- moved C1 0.55 mm to (118.2, 78.5)
- moved C2 0.15 mm to (125.5, 86.4)
Connections:
- U1 pad 10: unconnected-(U1-Pad10) -> col9
- U1 pad 11: unconnected-(U1-Pad11) -> col10
- U1 pad 17: unconnected-(U1-Pad17) -> col2
- U1 pad 18: unconnected-(U1-Pad18) -> col1
- U1 pad 19: unconnected-(U1-Pad19) -> col0
- U1 pad 20: unconnected-(U1-Pad20) -> row0
- U1 pad 21: unconnected-(U1-Pad21) -> row1
- U1 pad 22: unconnected-(U1-Pad22) -> row2
- U1 pad 23: unconnected-(U1-Pad23) -> col3
- U1 pad 25: unconnected-(U1-Pad25) -> col4
- U1 pad 26: unconnected-(U1-Pad26) -> col5
- U1 pad 7: unconnected-(U1-Pad7) -> col6
- U1 pad 8: unconnected-(U1-Pad8) -> col7
- U1 pad 9: unconnected-(U1-Pad9) -> col8
Routing:
- net col10: track 59.8 -> 205.5 mm
- net row0: track 196.1 -> 319.5 mm
- net col9: track 69.1 -> 166.1 mm, vias 0 -> 1
- net row1: track 200.8 -> 293.3 mm
- net col0: track 55.7 -> 147.6 mm
- net col8: track 66.8 -> 139.3 mm, vias 0 -> 1
- net col1: track 60.4 -> 127.7 mm
- net col7: track 39.6 -> 103.7 mm, vias 0 -> 1
- net col2: track 60.3 -> 108.7 mm
- net col6: track 39.6 -> 85.7 mm, vias 0 -> 1
- net col3: track 39.6 -> 67.5 mm, vias 0 -> 1
- net row2: track 200.7 -> 226.4 mm
- net col5: track 57.5 -> 77.2 mm, vias 0 -> 1
- net col4: track 39.6 -> 51.7 mm, vias 0 -> 1
- net GND: track 1.33 -> 9.89 mm, vias 1 -> 3
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
Commit message: Production files added
Parts:
- removed SW33b1: SW_Push, mbk:Choc-1.25u-solder
- removed SW34b1: SW_Push, mbk:Choc-1u-solder
- moved D33 2.30 mm to (214.2, 73.4)
Routing:
- net Net-(D33-Pad2): track 5.35 -> 3.05 mm
- net col9: track 166.1 -> 163.9 mm
- net Net-(D34-Pad2): track 5.35 -> 3.10 mm
