File: Switch Plate/Choc40-switch_plate.kicad_sch (KiCad schematic)
At the start: 42 parts, among them SW1 SW_Push, SW10 SW_Push, SW11 SW_Push, SW12 SW_Push, SW13 SW_Push, SW14 SW_Push, SW15 SW_Push, SW16 SW_Push, SW17 SW_Push, SW18 SW_Push, SW19 SW_Push, SW2 SW_Push, SW20 SW_Push, SW21 SW_Push, SW22 SW_Push, SW23 SW_Push, SW24 SW_Push, SW25 SW_Push, SW26 SW_Push, SW27 SW_Push, SW28 SW_Push, SW29 SW_Push, SW3 SW_Push, SW30 SW_Push, SW31 SW_Push, SW32 SW_Push, SW33a1 SW_Push, SW33b1 SW_Push, SW34a1 SW_Push, SW34b1 SW_Push, SW35 SW_Push, SW36 SW_Push, SW37 SW_Push, SW38 SW_Push, SW39 SW_Push, SW4 SW_Push, SW40 SW_Push, SW5 SW_Push, SW6 SW_Push, SW7 SW_Push, SW8 SW_Push, SW9 SW_Push

Commit message: Production files added
Parts:
- removed SW33b1: SW_Push, mbk:Choc-1.25u-solder, symbol Switch:SW_Push
- removed SW34b1: SW_Push, mbk:Choc-1u-solder, symbol Switch:SW_Push
- added H1, H2, H3, H4: MountingHole, MountingHole:MountingHole_2.2mm_M2, symbol Mechanical:MountingHole
- SW1, SW10, SW11, SW12, SW14, SW15, SW16, SW17, SW18, SW19, SW2, SW20, SW21, SW22, SW25, SW26, SW27, SW28, SW29, SW3, SW30, SW31, SW32, SW33a1, SW36, SW37, SW4, SW5, SW6, SW7, SW8, SW9: footprint mbk:Choc-1u-solder -> mbk:Choc-1u-cutout
- SW13, SW34a1, SW35, SW39, SW40: footprint mbk:Choc-1.25u-solder -> mbk:Choc-1u-cutout
- SW23, SW24: footprint mbk:Choc-1.75u-solder -> mbk:Choc-1u-cutout
- SW38: footprint mbk:Choc-6.25u-solder -> mbk:Choc-6.25u-cutout
